File: board.sch (EAGLE design)
At the start: 26 parts, among them IC1 74HCT125D, J1 M5STICK_PINOUT, J2 JST-SH 4 Position Connector, J3 USB_A_PTH_MALE

Commit message: fixed silkscreen for all components
Parts:
- removed D1, D2, D3, D4, D5, D6, D7, D8: APA102-5050, SparkFun-LED:APA102-5050
- added 1, 2, 3, 4, 5, 6, 7, 8: APA102-5050, SparkFun-LED:APA102-5050
- C1, C2, C3, C4, C5, C6, C7, C8, C9: value (none) -> 0.1uF
- J5: value (none) -> SERIAL
- R1: value (none) -> 330
- S1: value (none) -> FLASH
- U1: value (none) -> M5STAMP PICO
Connections:
- net CI$1: now also 1.CI; no longer D1.CI
- net CI$2: now also 1.CO, 2.CI; no longer D1.CO, D2.CI
- net CI$3: now also 2.CO, 3.CI; no longer D2.CO, D3.CI
- net CI$4: now also 3.CO, 4.CI; no longer D3.CO, D4.CI
- net CI$5: now also 4.CO, 5.CI; no longer D4.CO, D5.CI
- net CI$6: now also 5.CO, 6.CI; no longer D5.CO, D6.CI
- net CI$7: now also 6.CO, 7.CI; no longer D6.CO, D7.CI
- net CI$8: now also 7.CO, 8.CI; no longer D7.CO, D8.CI
- net CO: now also 8.CO; no longer D8.CO
- net DI$1: now also 1.DI; no longer D1.DI
- net DI$2: now also 1.DO, 2.DI; no longer D1.DO, D2.DI
- net DI$3: now also 2.DO, 3.DI; no longer D2.DO, D3.DI
- net DI$4: now also 3.DO, 4.DI; no longer D3.DO, D4.DI
- net DI$5: now also 4.DO, 5.DI; no longer D4.DO, D5.DI
- net DI$6: now also 5.DO, 6.DI; no longer D5.DO, D6.DI
- net DI$7: now also 6.DO, 7.DI; no longer D6.DO, D7.DI
- net DI$8: now also 7.DO, 8.DI; no longer D7.DO, D8.DI
- net DO: now also 8.DO; no longer D8.DO
- net GND: now also 1.GND, 2.GND, 3.GND, 4.GND, 5.GND, 6.GND, 7.GND, 8.GND; no longer D1.GND, D2.GND, D3.GND, D4.GND, D5.GND, D6.GND, D7.GND, D8.GND
- net VCC: now also 1.VCC, 2.VCC, 3.VCC, 4.VCC, 5.VCC, 6.VCC, 7.VCC, 8.VCC; no longer D1.VCC, D2.VCC, D3.VCC, D4.VCC, D5.VCC, D6.VCC, D7.VCC, D8.VCC
